File: pcbs/8view/8view.kicad_pcb (KiCad board)
At the start: 4 copper layers, 25.9 x 35.6 mm, 49 parts, among them J1 Conn_01x10_Female, J2 Conn_01x10_Female, J3 Conn_01x06_Female, J4 Conn_01x06_Female, U1 ATtiny828-A, U2 HDSP-A151, U3 HDSP-A151

Commit message: 8view: flipped mode
Connections:
- net Net-(R11-Pad2) renamed /D1_O1
- net Net-(R12-Pad2) renamed /D1_O2
- net Net-(R13-Pad2) renamed /D1_O3
- net Net-(R14-Pad2) renamed /D1_O4
- net Net-(R15-Pad2) renamed /D1_O5
- net Net-(R16-Pad2) renamed /D1_O6
- net Net-(R17-Pad2) renamed /D1_O7
- net Net-(R18-Pad2) renamed /D1_O8
- net Net-(R19-Pad2) renamed /D2_O1
- net Net-(R20-Pad2) renamed /D2_O2
- net Net-(R21-Pad2) renamed /D2_O3
- net Net-(R22-Pad2) renamed /D2_O4
- net Net-(R23-Pad2) renamed /D2_O5
- net Net-(R24-Pad2) renamed /D2_O6
- net Net-(R25-Pad2) renamed /D2_O7
- net Net-(R26-Pad2) renamed /D2_O8
